Commit message: geomagic: corrected touchx urdf

File: geomagic/touchx_description/urdf/touch_x.urdf (robot description, URDF)
Before this commit: robot geomagic_touch, 7 links, 6 joints
Joints:
- joint j1: origin xyz=0 0 0.09 rpy=0 0 0 -> xyz=0 0 0.05499100 rpy=0 0 0
- joint j2: origin xyz=-0.0075 0 0.035 rpy=0 0 0 -> xyz=0.02053590 0 0.05108434 rpy=0 0 0
- joint j3: axis 1 0 0 -> -1 0 0; origin xyz=0.0075 .134 0 rpy=-1.5 0 0 -> xyz=-0.01079507 -0.09921078 0.08910355 rpy=0 0 0
- joint j4: origin xyz=0 0.08 0 -> xyz=-0.00939800 -0.09969500 0 rpy=0 0 0
- joint j5: origin xyz=0 0.0525 0 rpy=0.5 0 0 -> xyz=-0.00184288 -0.03289300 0 rpy=0 0 0
- joint j6: origin xyz=0 -0.023 0 rpy=3.14159 3.14159 0 -> xyz=0.00001888 -0.02817081 -0.00970118 rpy=0 0 0
