Commit message: Moved touchx_description files into geomagic_description

File: geomagic/geomagic_description/urdf/touch.urdf (robot description, URDF)
Before this commit: robot geomagic_touch, 7 links, 6 joints
Links:
- removed link lower_wrist
- removed link upper_wrist
- added link tip; visual mesh filename=package://geomagic_description/meshes/touch/tip.stl
- added link wrist; visual mesh filename=package://geomagic_description/meshes/touch/wrist.stl
- link base: geometry visual mesh filename=package://geomagic_description/meshes/touch/base.stl
- link lower_arm: geometry visual mesh filename=package://geomagic_description/meshes/touch/lower_arm.stl
- link stylus: geometry visual mesh filename=package://geomagic_description/meshes/touch/pen.stl
- link torso: geometry visual mesh filename=package://geomagic_description/meshes/touch/torso.stl
- link upper_arm: geometry visual mesh filename=package://geomagic_description/meshes/touch/upper_arm.stl
Joints:
- joint j1: origin xyz=0 0 0.05499100 rpy=0 0 0 -> xyz=0 0 0.09 rpy=0 0 0
- joint j2: origin xyz=0.02053590 0 0.05108434 rpy=0 0 0 -> xyz=-0.0075 0 0.035 rpy=0 0 0
- joint j3: axis -1 0 0 -> 1 0 0; origin xyz=-0.01079507 -0.09921078 0.08910355 rpy=0 0 0 -> xyz=0.0075 .134 0 rpy=-1.5 0 0
- joint j4: child upper_wrist -> wrist; origin xyz=-0.00939800 -0.09969500 0 rpy=0 0 0 -> xyz=0 0.08 0
- joint j5: child lower_wrist -> tip; origin xyz=-0.00184288 -0.03289300 0 rpy=0 0 0 -> xyz=0 0.0525 0 rpy=0.5 0 0; parent upper_wrist -> wrist
- joint j6: origin xyz=0.00001888 -0.02817081 -0.00970118 rpy=0 0 0 -> xyz=0 -0.023 0 rpy=3.14159 3.14159 0; parent lower_wrist -> tip

File: geomagic/geomagic_description/urdf/touch_x.urdf (robot description, URDF)
Before this commit: robot geomagic_touch, 7 links, 6 joints
Links:
- removed link tip
- removed link wrist
- added link lower_wrist; visual mesh filename=package://geomagic_description/meshes/touch_x/lower_wrist.s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
- added link upper_wrist; visual mesh filename=package://geomagic_description/meshes/touch_x/upper_wrist.s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
- link base: geometry visual mesh filename=package://geomagic_description/meshes/touch_x/base.stl
- link lower_arm: geometry visual mesh filename=package://geomagic_description/meshes/touch_x/lower_arm.stl
- link stylus: geometry visual mesh filename=package://geomagic_description/meshes/touch_x/stylus.stl
- link torso: geometry visual mesh filename=package://geomagic_description/meshes/touch_x/torso.stl
- link upper_arm: geometry visual mesh filename=package://geomagic_description/meshes/touch_x/upper_arm.stl
Joints:
- removed joint elbow
- removed joint pitch
- removed joint roll
- removed joint shoulder
- removed joint waist
- removed joint yaw
- added joint j1: type revolute, parent base, child torso, origin xyz=0 0 0.05499100 rpy=0 0 0, axis 0 0 -1, limit lower=-0.98 upper=0.98 effort=5 velocity=100
- added joint j2: type revolute, parent torso, child upper_arm, origin xyz=0.02053590 0 0.05108434 rpy=0 0 0, axis -1 0 0, limit lower=0 upper=1.75 effort=5 velocity=100
- added joint j3: type revolute, parent upper_arm, child lower_arm, origin xyz=-0.01079507 -0.09921078 0.08910355 rpy=0 0 0, axis -1 0 0, limit lower=-0.81 upper=1.25 effort=5 velocity=100
- added joint j4: type revolute, parent lower_arm, child upper_wrist, origin xyz=-0.00939800 -0.09969500 0 rpy=0 0 0, axis 0 1 0, limit lower=3.92 upper=8.83 effort=5 velocity=100
- added joint j5: type revolute, parent upper_wrist, child lower_wrist, origin xyz=-0.00184288 -0.03289300 0 rpy=0 0 0, axis 1 0 0, limit lower=-0.5 upper=1.75 effort=5 velocity=100
- added joint j6: type revolute, parent lower_wrist, child stylus, origin xyz=0.00001888 -0.02817081 -0.00970118 rpy=0 0 0, axis 0 1 0, limit lower=-2.58 upper=2.58 effort=5 velocity=100
